File: pcb/popnmusic.kicad_pcb (KiCad board)
At the start: 2 copper layers, 321.5 x 121.4 mm, 10 parts, among them SW1 SW_Push, SW2 SW_Push, SW3 SW_Push, SW4 SW_Push, SW5 SW_Push, SW6 SW_Push, SW7 SW_Push, SW8 SW_Push, SW9 SW_Push, U1 XIAO-RP2040-DIP

Commit message: Add files via upload
Parts:
- added J1: Conn_01x02, Connector_PinHeader_2.54mm:PinHeader_1x02_P2.54mm_Vertical, F.Cu at (135.0, 39.0)
- added J10: Conn_01x02, Connector_PinHeader_2.54mm:PinHeader_1x02_P2.54mm_Vertical, F.Cu at (139.0, 72.0)
- added J11: Conn_01x02, Connector_PinHeader_2.54mm:PinHeader_1x02_P2.54mm_Vertical, F.Cu at (139.0, 98.0)
- added J12: Conn_01x02, Connector_PinHeader_2.54mm:PinHeader_1x02_P2.54mm_Vertical, F.Cu at (221.0, 54.2)
- added J13: Conn_01x02, Connector_PinHeader_2.54mm:PinHeader_1x02_P2.54mm_Vertical, F.Cu at (162.0, 72.0)
- added J14: Conn_01x02, Connector_PinHeader_2.54mm:PinHeader_1x02_P2.54mm_Vertical, F.Cu at (161.0, 98.0)
- added J15: Conn_01x02, Connector_PinHeader_2.54mm:PinHeader_1x02_P2.54mm_Vertical, F.Cu at (219.5, 81.9)
- added J16: Conn_01x02, Connector_PinHeader_2.54mm:PinHeader_1x02_P2.54mm_Vertical, F.Cu at (184.5, 72.0)
- added J17: Conn_01x02, Connector_PinHeader_2.54mm:PinHeader_1x02_P2.54mm_Vertical, F.Cu at (183.5, 98.0)
- added J18: Conn_01x02, Connector_PinHeader_2.54mm:PinHeader_1x02_P2.54mm_Vertical, F.Cu at (209.6, 117.5)
- added J2: Conn_01x02, Connector_PinHeader_2.54mm:PinHeader_1x02_P2.54mm_Vertical, F.Cu at (135.0, 46.0)
- added J3: Conn_01x02, Connector_PinHeader_2.54mm:PinHeader_1x02_P2.54mm_Vertical, F.Cu at (135.0, 53.0)
- added J4: Conn_01x02, Connector_PinHeader_2.54mm:PinHeader_1x02_P2.54mm_Vertical, F.Cu at (135.0, 60.0)
- added J5: Conn_01x02, Connector_PinHeader_2.54mm:PinHeader_1x02_P2.54mm_Vertical, F.Cu at (140.0, 60.0)
- added J6: Conn_01x02, Connector_PinHeader_2.54mm:PinHeader_1x02_P2.54mm_Vertical, F.Cu at (144.5, 60.5)
- added J7: Conn_01x02, Connector_PinHeader_2.54mm:PinHeader_1x02_P2.54mm_Vertical, F.Cu at (149.0, 60.5)
- added J8: Conn_01x02, Connector_PinHeader_2.54mm:PinHeader_1x02_P2.54mm_Vertical, F.Cu at (153.5, 60.5)
- added J9: Conn_01x02, Connector_PinHeader_2.54mm:PinHeader_1x02_P2.54mm_Vertical, F.Cu at (158.0, 60.2)
- added REF**: MountingHole_2.1mm, MountingHole:MountingHole_2.1mm, F.Cu at (163.5, 94.5)
- added REF**: MountingHole_2.1mm, MountingHole:MountingHole_2.1mm, F.Cu at (152.0, 108.5)
- added REF**: MountingHole_2.1mm, MountingHole:MountingHole_2.1mm, F.Cu at (211.0, 44.0)
- added REF**: MountingHole_2.1mm, MountingHole:MountingHole_2.1mm, F.Cu at (152.5, 82.0)
- added REF**: MountingHole_2.1mm, MountingHole:MountingHole_2.1mm, F.Cu at (197.0, 55.0)
- added REF**: MountingHole_2.1mm, MountingHole:MountingHole_2.1mm, F.Cu at (209.5, 68.0)
- added REF**: MountingHole_2.1mm, MountingHole:MountingHole_2.1mm, F.Cu at (223.5, 68.0)
- added REF**: MountingHole_2.1mm, MountingHole:MountingHole_2.1mm, F.Cu at (142.0, 68.0)
- added REF**: MountingHole_2.1mm, MountingHole:MountingHole_2.1mm, F.Cu at (197.0, 108.0)
- added REF**: MountingHole_2.1mm, MountingHole:MountingHole_2.1mm, F.Cu at (175.0, 108.5)
- added REF**: MountingHole_2.1mm, MountingHole:MountingHole_2.1mm, F.Cu at (164.0, 68.0)
- added REF**: MountingHole_2.1mm, MountingHole:MountingHole_2.1mm, F.Cu at (141.5, 95.0)
- added REF**: MountingHole_2.1mm, MountingHole:MountingHole_2.1mm, F.Cu at (223.0, 44.0)
- added REF**: MountingHole_2.1mm, MountingHole:MountingHole_2.1mm, F.Cu at (197.0, 82.0)
- added REF**: MountingHole_2.1mm, MountingHole:MountingHole_2.1mm, F.Cu at (186.5, 68.0)
- added REF**: MountingHole_2.1mm, MountingHole:MountingHole_2.1mm, F.Cu at (175.0, 81.5)
- added REF**: MountingHole_2.1mm, MountingHole:MountingHole_2.1mm, F.Cu at (209.0, 95.0)
- added REF**: MountingHole_2.1mm, MountingHole:MountingHole_2.1mm, F.Cu at (186.0, 94.5)
- added REF**: MountingHole_2.1mm, MountingHole:MountingHole_2.1mm, F.Cu at (223.0, 95.0)
- moved SW3 142.1 mm to (214.5, 58.5), turned to -90 degrees
- moved SW1 125.2 mm to (143.2, 78.4)
- moved SW2 89.5 mm to (142.8, 104.5)
- moved SW9 69.6 mm to (205.5, 111.1), turned to 180 degrees
- moved SW8 65.4 mm to (188.8, 104.5)
- moved SW7 50.8 mm to (188.6, 78.4)
- moved SW4 45.2 mm to (166.1, 78.4)
- moved SW6 33.1 mm to (213.1, 86.0), turned to -90 degrees
- moved SW5 24.5 mm to (165.3, 104.5)
- moved U1 1.89 mm to (148.0, 45.8)
Connections:
- SW1 pad 1: GND -> Net-(J10-Pin_2)
- SW1 pad 2: Net-(U1-GPIO26/ADC0/A0) -> Net-(J10-Pin_1)
- SW2 pad 1: GND -> Net-(J11-Pin_2)
- SW2 pad 2: Net-(U1-GPIO27/ADC1/A1) -> Net-(J11-Pin_1)
- SW3 pad 1: GND -> Net-(J12-Pin_2)
- SW3 pad 2: Net-(U1-GPIO28/ADC2/A2) -> Net-(J12-Pin_1)
- SW4 pad 1: GND -> Net-(J13-Pin_2)
- SW4 pad 2: Net-(U1-GPIO29/ADC3/A3) -> Net-(J13-Pin_1)
- SW5 pad 1: GND -> Net-(J14-Pin_2)
- SW5 pad 2: Net-(U1-GPIO6/SDA) -> Net-(J14-Pin_1)
- SW6 pad 1: GND -> Net-(J15-Pin_2)
- SW6 pad 2: Net-(U1-GPIO7/SCL) -> Net-(J15-Pin_1)
- SW7 pad 1: GND -> Net-(J16-Pin_2)
- SW7 pad 2: Net-(U1-GPIO0/TX) -> Net-(J16-Pin_1)
- SW8 pad 1: GND -> Net-(J17-Pin_2)
- SW8 pad 2: Net-(U1-GPIO1/RX) -> Net-(J17-Pin_1)
- SW9 pad 1: GND -> Net-(J18-Pin_2)
- SW9 pad 2: Net-(U1-GPIO2/SCK) -> Net-(J18-Pin_1)
- U1 pad 1: Net-(U1-GPIO26/ADC0/A0) -> Net-(J1-Pin_2)
- U1 pad 2: Net-(U1-GPIO27/ADC1/A1) -> Net-(J2-Pin_2)
- U1 pad 3: Net-(U1-GPIO28/ADC2/A2) -> Net-(J3-Pin_2)
- U1 pad 4: Net-(U1-GPIO29/ADC3/A3) -> Net-(J4-Pin_2)
- U1 pad 5: Net-(U1-GPIO6/SDA) -> Net-(J5-Pin_2)
- U1 pad 6: Net-(U1-GPIO7/SCL) -> Net-(J6-Pin_2)
- U1 pad 7: Net-(U1-GPIO0/TX) -> Net-(J7-Pin_2)
- U1 pad 8: Net-(U1-GPIO1/RX) -> Net-(J8-Pin_2)
- U1 pad 9: Net-(U1-GPIO2/SCK) -> Net-(J9-Pin_2)
Routing:
- net GND: track 593.0 -> 93.2 mm
- net Net-(U1-GPIO28/ADC2/A2): track 367.2 -> 0.00 mm
- net Net-(U1-GPIO0/TX): track 284.3 -> 0.00 mm
- net Net-(U1-GPIO2/SCK): track 196.3 -> 0.00 mm
- net Net-(U1-GPIO26/ADC0/A0): track 180.8 -> 0.00 mm
- net Net-(U1-GPIO27/ADC1/A1): track 121.2 -> 0.00 mm
- net Net-(U1-GPIO1/RX): track 115.8 -> 0.00 mm
- net Net-(U1-GPIO6/SDA): track 80.7 -> 0.00 mm
- net Net-(U1-GPIO29/ADC3/A3): track 51.1 -> 0.00 mm
- net Net-(U1-GPIO7/SCL): track 30.6 -> 0.00 mm
- net Net-(J8-Pin_2): track 0.00 -> 30.3 mm
- net Net-(J9-Pin_2): track 0.00 -> 30.2 mm
- net Net-(J4-Pin_2): track 0.00 -> 27.9 mm
- net Net-(J3-Pin_2): track 0.00 -> 25.7 mm
- net Net-(J2-Pin_2): track 0.00 -> 23.9 mm
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Other:
- board size 321.5 x 121.4 mm -> 95.5 x 86 mm
- board text removed: "KONAMI presents the new sensation rhythm game. Pop'n Music! Let's enjoy the music together. It's time to be happy!"
