File: pcb/popnmusic.kicad_sch (KiCad schematic)
At the start: 10 parts, among them SW1 SW_Push, SW2 SW_Push, SW3 SW_Push, SW4 SW_Push, SW5 SW_Push, SW6 SW_Push, SW7 SW_Push, SW8 SW_Push, SW9 SW_Push, U1 XIAO-RP2040-DIP

Commit message: Add files via upload
Parts:
- added J1, J10, J11, J12, J13, J14, J15, J16, J17, J18, J2, J3, J4, J5, J6, J7, J8, J9: Conn_01x02, Connector_PinHeader_2.54mm:PinHeader_1x02_P2.54mm_Vertical, symbol Connector_Generic:Conn_01x02
Connections:
- net GND: now also J1.1 (Pin_1), J2.1 (Pin_1), J3.1 (Pin_1), J4.1 (Pin_1), J5.1 (Pin_1), J6.1 (Pin_1), J7.1 (Pin_1), J8.1 (Pin_1), J9.1 (Pin_1); no longer SW1.1, SW2.1, SW3.1, SW4.1, SW5.1, SW6.1, SW7.1, SW8.1, SW9.1
- net at SW4.2: now also J13.1 (Pin_1); no longer U1.4 (GPIO29/ADC3/A3)
- net at SW3.2: now also J12.1 (Pin_1); no longer U1.3 (GPIO28/ADC2/A2)
- net at SW6.2: now also J15.1 (Pin_1); no longer U1.6 (GPIO7/SCL)
- net at U1.1 (GPIO26/ADC0/A0): now also J1.2 (Pin_2); no longer SW1.2
- net at U1.2 (GPIO27/ADC1/A1): now also J2.2 (Pin_2); no longer SW2.2
- net at SW7.2: now also J16.1 (Pin_1); no longer U1.7 (GPIO0/TX)
- net at SW5.2: now also J14.1 (Pin_1); no longer U1.5 (GPIO6/SDA)
- net at SW8.2: now also J17.1 (Pin_1); no longer U1.8 (GPIO1/RX)
- net at SW9.2: now also J18.1 (Pin_1); no longer U1.9 (GPIO2/SCK)
- new net: J15.2 (Pin_2), SW6.1
- new net: J6.2 (Pin_2), U1.6 (GPIO7/SCL)
- new net: J12.2 (Pin_2), SW3.1
- new net: J10.1 (Pin_1), SW1.2
- new net: J10.2 (Pin_2), SW1.1
- new net: J18.2 (Pin_2), SW9.1
- new net: J14.2 (Pin_2), SW5.1
- new net: J16.2 (Pin_2), SW7.1
- new net: J13.2 (Pin_2), SW4.1
- new net: J3.2 (Pin_2), U1.3 (GPIO28/ADC2/A2)
- new net: J5.2 (Pin_2), U1.5 (GPIO6/SDA)
- new net: J17.2 (Pin_2), SW8.1
- new net: J4.2 (Pin_2), U1.4 (GPIO29/ADC3/A3)
- new net: J7.2 (Pin_2), U1.7 (GPIO0/TX)
- new net: J8.2 (Pin_2), U1.8 (GPIO1/RX)
- new net: J9.2 (Pin_2), U1.9 (GPIO2/SCK)
- new net: J11.2 (Pin_2), SW2.1
- new net: J11.1 (Pin_1), SW2.2
